File: pcbs/relay-attentuator-SMD.sch (EAGLE design)
At the start: 71 parts, among them IC1 MCP23S17SO, IC2 ULN2803, IC3 ULN2803, K1 IM43TS, K2 IM43TS, K3 IM43TS, K4 IM43TS, K5 IM43TS, K6 IM43TS, K7 IM43TS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

Commit message: new designs
Parts:
- removed IC1: MCP23S17SO, microchip:MCP23S17SO
- removed IN, OUT: 22-23-2031, con-molex:22-23-2031
- removed LED: (no value), led:LEDCHIPLED_1206
- removed LOGO1: OSHW_LOGO_FILLX0200-NT, ohw-logo:OSHW_LOGO_FILLX0200-NT
- removed RLED: 2.4k, rcl:R-EU_R1206
- removed X1: 22-23-2051, con-molex:22-23-2051
- added J1, J2: B4B-XH-A, B4B-XH-A:B4B-XH-A
- added J3, J4: B3B-XH-A, B3B-XH-A:B3B-XH-A
- added R17, R18, R19, R20, R21: 47R, rcl:R-EU_R1206
- added S1: 2454982-2, 2454982-2:2454982-2
- added U1: MCP23017-E/SO, MCP23017-E_SO:MCP23017-E/SO
- C1: device rcl:C-EUC1206 -> rcl:CPOL-EUE3.5-8
- C3: device rcl:CPOL-EUE3.5-8 -> rcl:C-EUC1206
Connections:
- removed net ATT_INL: IN-1.S, K12.S, R1A.1
- removed net CS: IC1.!CS, X1-3.S
- removed net N$67: LED.C, RLED.1
- removed net SCK: IC1.SCK, X1-2.S
- removed net SI: IC1.SI, X1-1.S
- new net N$49: J3.3, K12.S, R1A.1
- new net N$55: R18.2, S1.NO_3, U1.A0
- new net N$56: R19.2, S1.NO_2, U1.A1
- new net N$57: R17.2, S1.NO_1, U1.A2
- new net N$58: J1.3, J2.3, R20.1, U1.SDA
- new net N$59: J1.4, J2.4, R21.1, U1.SCK
- net +5V: now also C1.+, C3.1, J1.2, J2.2, R20.2, R21.2, S1.COM_1, S1.COM_2, S1.COM_3, U1.!RESET, U1.VDD; no longer C1.1, C3.+, IC1.!RESET, IC1.VDD, LED.A, X1-4.S
- net AGND: now also J3.2, J4.2; no longer IN-2.S, OUT-2.S
- net ATT_INR: now also J3.1; no longer IN-3.S
- net DGND: now also C1.-, C3.2, J1.1, J2.1, R17.1, R18.1, R19.1, U1.VSS; no longer C1.2, C3.-, IC1.A0, IC1.A1, IC1.A2, IC1.VSS, RLED.2, X1-5.S
- net N$1: now also IC3.O1; no longer IC2.O8
- net N$10: now also IC3.O2; no longer IC2.O7
- net N$11: now also IC3.O3; no longer IC2.O6
- net N$12: now also IC3.O4; no longer IC2.O5
- net N$13: now also IC3.O5; no longer IC2.O4
- net N$14: now also IC3.O6; no longer IC2.O3
- net N$15: now also IC3.O7; no longer IC2.O2
- net N$16: now also IC3.O8; no longer IC2.O1
- net N$18: now also IC2.O7; no longer IC3.O7
- net N$19: now also IC2.O3; no longer IC3.O3
- net N$2: now also IC2.O8; no longer IC3.O8
- net N$20: now also IC2.O4; no longer IC3.O4
- net N$3: now also IC2.O2; no longer IC3.O2
- net N$33: now also IC2.I8, U1.GPB7; no longer IC1.GPA7, IC2.I1
- net N$34: now also IC2.I7, U1.GPB6; no longer IC1.GPA6, IC2.I2
- net N$35: now also IC2.I6, U1.GPB5; no longer IC1.GPA5, IC2.I3
- net N$36: now also IC2.I5, U1.GPB4; no longer IC1.GPA4, IC2.I4
- net N$37: now also IC2.I4, U1.GPB3; no longer IC1.GPA3, IC2.I5
- net N$38: now also IC2.I3, U1.GPB2; no longer IC1.GPA2, IC2.I6
- net N$39: now also IC2.I2, U1.GPB1; no longer IC1.GPA1, IC2.I7
- net N$4: now also IC2.O6; no longer IC3.O6
- net N$40: now also IC2.I1, U1.GPB0; no longer IC1.GPA0, IC2.I8
- net N$41: now also U1.GPA0; no longer IC1.GPB7
- net N$42: now also U1.GPA1; no longer IC1.GPB6
- net N$43: now also U1.GPA2; no longer IC1.GPB5
- net N$44: now also U1.GPA3; no longer IC1.GPB4
- net N$45: now also U1.GPA4; no longer IC1.GPB3
- net N$46: now also U1.GPA5; no longer IC1.GPB2
- net N$47: now also U1.GPA6; no longer IC1.GPB1
- net N$48: now also U1.GPA7; no longer IC1.GPB0
- net N$5: now also IC2.O5; no longer IC3.O5
- net N$69: now also J4.3; no longer OUT-3.S
- net N$71: now also J4.1; no longer OUT-1.S
- net N$9: now also IC2.O1; no longer IC3.O1
Other:
- moved on the sheet: C2, C4, IC2, IC3

Commit message: fixes
Connections:
- net +5V: now also R17.1, R18.1, R19.1; no longer S1.COM_1, S1.COM_2, S1.COM_3
- net DGND: now also S1.COM_1, S1.COM_2, S1.COM_3; no longer R17.1, R18.1, R19.1
