File: pcbs/relay-attentuator-THRU.brd (EAGLE design)
At the start: 98.7 x 50.5 mm, 75 parts, among them IC2 ULN2803, IC3 ULN2803, J1 B4B-XH-A, J2 B4B-XH-A, J3 B3B-XH-A, J4 B3B-XH-A, K1 IM43TS, K2 IM43TS, K3 IM43TS, K4 IM43TS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

Commit message: fixes
Parts:
- moved R21 6.24 mm to (20.3, 35.6), turned to 180 degrees
- moved R20 2.73 mm to (25.7, 35.6), turned to 0 degrees
Connections:
- net +5V: now also R17.1, R18.1, R19.1; no longer S1.1, S1.2, S1.3
- net DGND: now also S1.1, S1.2, S1.3; no longer R17.1, R18.1, R19.1
Routing:
- net +5V: track 202.7 -> 214.1 mm
- net N$58: track 38.0 -> 34.9 mm
- net N$59: track 33.6 -> 32.2 mm
- net N$45: track 12.1 -> 11.5 mm
- net N$48: track 18.0 -> 17.5 mm
- net N$47: track 15.6 -> 15.1 mm
- net N$44: track 10.2 -> 9.66 mm
- net N$46: track 13.8 -> 13.3 mm
